File: 回路-基板/master/master.kicad_sch (KiCad schematic)
At the start: 23 parts, among them J1 Ext. PWR, J2 Conn_01x07_Pin, SW1 SW_SPDT, SW2 SW_SPDT, SW3 RESET, U1 TWE-L-DP-W, U2 LM1117MP-3.3, U3 DEV-16771

Commit message: 再度フットプリント関連付けした
Parts:
- SW1, SW2: footprint (none) -> @2024-cansat:SS12D01G4
Changed lines of the file:
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@@
 			)
 		)
-		(property "Footprint" ""
+		(property "Footprint" "@2024-cansat:SS12D01G4"
 			(at 187.96 135.89 0)
 			(effects
@@
 			)
 		)
-		(property "Footprint" ""
+		(property "Footprint" "@2024-cansat:SS12D01G4"
 			(at 187.96 153.67 0)
 			(effects

Commit message: PCB_1
Parts:
- SW1, SW2: footprint @2024-cansat:SS12D01G4 -> 2024-cansat:SS12D01G4
- SW3: footprint @2024-cansat:TVBP06-B043C -> 2024-cansat:TVBP06-B043C
- U3: footprint @2024-cansat:MODULE_DEV-16771 -> 2024-cansat:MODULE_DEV-16771
- U4: footprint @2024-cansat:Display -> 2024-cansat:Display
Changed lines of the file:
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@@
 			)
 		)
-		(property "Footprint" "@2024-cansat:MODULE_DEV-16771"
+		(property "Footprint" "2024-cansat:MODULE_DEV-16771"
 			(at 133.35 81.28 0)
 			(effects
@@
 			)
 		)
-		(property "Footprint" "@2024-cansat:TVBP06-B043C"
+		(property "Footprint" "2024-cansat:TVBP06-B043C"
 			(at 194.31 36.83 0)
 			(effects
@@
 			)
 		)
-		(property "Footprint" "@2024-cansat:SS12D01G4"
+		(property "Footprint" "2024-cansat:SS12D01G4"
 			(at 187.96 135.89 0)
 			(effects
@@
 			)
 		)
-		(property "Footprint" "@2024-cansat:Display"
+		(property "Footprint" "2024-cansat:Display"
 			(at 191.77 60.198 0)
 			(effects
@@
 			)
 		)
-		(property "Footprint" "@2024-cansat:SS12D01G4"
+		(property "Footprint" "2024-cansat:SS12D01G4"
 			(at 187.96 153.67 0)
 			(effects

Commit message: PCB進めた
発注用ファイルも作成した
Parts:
- R1, R2, R3, R4, R5, R6, R7, R8: footprint Resistor_SMD:R_0603_1608Metric -> Resistor_THT:R_Axial_DIN0207_L6.3mm_D2.5mm_P7.62mm_Horizontal
Changed lines of the file:
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@@
 			)
 		)
-		(property "Footprint" "Resistor_SMD:R_0603_1608Metric"
+		(property "Footprint" "Resistor_THT:R_Axial_DIN0207_L6.3mm_D2.5mm_P7.62mm_Horizontal"
 			(at 180.34 95.25 0)
 			(effects
@@
 			)
 		)
-		(property "Footprint" "Resistor_SMD:R_0603_1608Metric"
+		(property "Footprint" "Resistor_THT:R_Axial_DIN0207_L6.3mm_D2.5mm_P7.62mm_Horizontal"
 			(at 198.12 128.27 0)
 			(effects
@@
 			)
 		)
-		(property "Footprint" "Resistor_SMD:R_0603_1608Metric"
+		(property "Footprint" "Resistor_THT:R_Axial_DIN0207_L6.3mm_D2.5mm_P7.62mm_Horizontal"
 			(at 198.12 146.05 0)
 			(effects
@@
 			)
 		)
-		(property "Footprint" "Resistor_SMD:R_0603_1608Metric"
+		(property "Footprint" "Resistor_THT:R_Axial_DIN0207_L6.3mm_D2.5mm_P7.62mm_Horizontal"
 			(at 45.72 144.78 0)
 			(effects
@@
 			)
 		)
-		(property "Footprint" "Resistor_SMD:R_0603_1608Metric"
+		(property "Footprint" "Resistor_THT:R_Axial_DIN0207_L6.3mm_D2.5mm_P7.62mm_Horizontal"
 			(at 182.88 95.25 0)
 			(effects
@@
 			)
 		)
-		(property "Footprint" "Resistor_SMD:R_0603_1608Metric"
+		(property "Footprint" "Resistor_THT:R_Axial_DIN0207_L6.3mm_D2.5mm_P7.62mm_Horizontal"
 			(at 130.81 151.13 0)
 			(effects
@@
 			)
 		)
-		(property "Footprint" "Resistor_SMD:R_0603_1608Metric"
+		(property "Footprint" "Resistor_THT:R_Axial_DIN0207_L6.3mm_D2.5mm_P7.62mm_Horizontal"
 			(at 186.69 36.83 0)
 			(effects
@@
 			)
 		)
-		(property "Footprint" "Resistor_SMD:R_0603_1608Metric"
+		(property "Footprint" "Resistor_THT:R_Axial_DIN0207_L6.3mm_D2.5mm_P7.62mm_Horizontal"
 			(at 130.81 157.48 0)
 			(effects
